File: Eagle Files/snow depth gauge 2B.brd (EAGLE design)
At the start: 47 x 48.3 mm, 30 parts, among them Q1 MMBT2222A, Q2 MMBT4403LT1SMD, Q3 MMBT2222A, Q4 MMBT2222A, U1 TEENSY 3.1, U2 XBEE-1B1

Commit message: PCB Ver. 2B Voltage Divider Update
Updated voltage divider components and values for measuring external 4.2
VDC LiPo battery.
Parts:
- R3: value 11K -> 10K
- R4: value 20K -> 27K
Changed lines of the file:
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@@
 <attribute name="PARTNO" value="KTR18EZPJ103" x="26.67" y="21.59" size="1.778" layer="27" rot="R180" display="off"/>
 </element>
-<element name="R4" library="resistor" package="R3216" value="20K" x="26.67" y="11.43" smashed="yes" rot="R180">
+<element name="R4" library="resistor" package="R3216" value="27K" x="26.67" y="11.43" smashed="yes" rot="R180">
 <attribute name="NAME" x="30.44825" y="11.39825" size="1.27" layer="25" rot="R180" align="center"/>
 <attribute name="VALUE" x="28.067" y="13.843" size="1.27" layer="27" rot="R180"/>
-<attribute name="PARTNO" value="KTR18EZPF2002" x="26.67" y="11.43" size="1.778" layer="27" rot="R180" display="off"/>
+<attribute name="PARTNO" value="KTR18EZPJ273" x="26.67" y="11.43" size="1.778" layer="27" rot="R180" display="off"/>
 </element>
 <element name="Q3" library="transistor-neu-to92" package="SOT23-BEC" value="MMBT2222A" x="26.67" y="33.02" smashed="yes" rot="R180">
@@
 <element name="U$3" library="SparkFun-Electromechanical" package="STAND-OFF" value="" x="44.45" y="2.54"/>
 <element name="U$4" library="SparkFun-Electromechanical" package="STAND-OFF" value="" x="44.45" y="45.72"/>
-<element name="R3" library="resistor" package="R3216" value="11K" x="26.67" y="13.97" smashed="yes" rot="R180">
+<element name="R3" library="resistor" package="R3216" value="10K" x="26.67" y="13.97" smashed="yes" rot="R180">
 <attribute name="NAME" x="30.44825" y="13.93825" size="1.27" layer="25" rot="R180" align="center"/>
 <attribute name="VALUE" x="28.067" y="16.383" size="1.27" layer="27" rot="R180"/>
-<attribute name="PARTNO" value="KTR18EZPF1102" x="26.67" y="13.97" size="1.778" layer="27" rot="R180" display="off"/>
+<attribute name="PARTNO" value="KTR18EZPJ103" x="26.67" y="13.97" size="1.778" layer="27" rot="R180" display="off"/>
 </element>
 <element name="U2" library="SparkFun-RF" package="XBEE-1" value="XBEE-1B1" x="33.02" y="12.7" smashed="yes">
